File: Eagle Schematics/DoorBell.brd (EAGLE design)
At the start: 43.5 x 17.8 mm, 9 parts, among them T1 2N3906

Commit message: Improved Board Labels
Parts:
- added C2: 1u, rcl:C025-025X050
- moved C1 3.81 mm to (35.6, 14.0)
- moved JP3 1.27 mm to (14.0, 10.2)
- moved R4 1.27 mm to (8.89, 10.2)
Connections:
- net GND: now also C2.2
- net SIG: now also C2.1
Routing:
- net GND: track 45.3 -> 53.6 mm
- net SIG: track 8.26 -> 13.3 mm
- net VCC: track 19.7 -> 21.3 mm
- net N$4: track 3.81 -> 2.54 mm
- net N$1: track 11.2 -> 10.2 mm
Other:
- board text added: "COM"
- board text added: "GND"
- board text added: "NO"
- board text added: "SIG"
- board text added: "TEST"
- board text added: "VCC"
Changed lines of the file:
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@@
 <plain>
 <wire x1="0" y1="0" x2="43.485" y2="0" width="0" layer="20"/>
-<wire x1="43.485" y1="0" x2="43.485" y2="17.77" width="0" layer="20"/>
 <wire x1="43.485" y1="17.77" x2="0" y2="17.77" width="0" layer="20"/>
 <wire x1="0" y1="17.77" x2="0" y2="0" width="0" layer="20"/>
+<text x="40.005" y="17.145" size="1.016" layer="25" rot="R270">VCC</text>
+<text x="40.005" y="5.715" size="1.016" layer="25" rot="R270">GND</text>
+<text x="41.91" y="10.795" size="1.016" layer="25" rot="R270">SIG</text>
+<wire x1="43.485" y1="0" x2="43.485" y2="17.77" width="0" layer="20"/>
+<text x="3.175" y="17.145" size="1.016" layer="25" rot="R270">NO</text>
+<text x="5.715" y="9.525" size="1.016" layer="25" rot="R270">TEST</text>
+<text x="3.175" y="5.715" size="1.016" layer="25" rot="R270">COM</text>
 </plain>
 <attributes>
@@
 <element name="R3" library="resistor" package="0204/5" value="10k" x="29.21" y="10.16"/>
 <element name="JP2" library="pinhead" package="1X03" value="TO RELAY" x="3.81" y="10.16" rot="R270"/>
-<element name="C1" library="rcl" package="C025-025X050" value="1u" x="35.56" y="10.16" rot="R270"/>
+<element name="C1" library="rcl" package="C025-025X050" value="1u" x="35.56" y="13.97" rot="R270"/>
 <element name="T1" library="transistor-neu-to92" package="TO92-EBC" value="2N3906" x="22.86" y="10.16" rot="R270"/>
 <element name="R1" library="resistor" package="0204/5" value="10k" x="29.21" y="5.08" rot="R180"/>
 <element name="R2" library="resistor" package="0204/5" value="10k" x="29.21" y="15.24"/>
-<element name="JP3" library="SparkFun-Connectors" package="1X01" value="M01PTH" x="15.24" y="10.16"/>
-<element name="R4" library="resistor" package="0204/5" value="10k" x="10.16" y="10.16" rot="R180"/>
+<element name="JP3" library="SparkFun-Connectors" package="1X01" value="M01PTH" x="13.97" y="10.16"/>
+<element name="R4" library="resistor" package="0204/5" value="10k" x="8.89" y="10.16" rot="R180"/>
+<element name="C2" library="rcl" package="C025-025X050" value="1u" x="35.56" y="3.81" rot="R270"/>
 </elements>
 <signals>
@@
 <contactref element="C1" pad="1"/>
 <contactref element="T1" pad="E"/>
-<wire x1="21.59" y1="12.7" x2="35.56" y2="12.7" width="0.4064" layer="1"/>
-<wire x1="35.56" y1="12.7" x2="40.005" y2="12.7" width="0.4064" layer="1"/>
-<wire x1="35.56" y1="11.43" x2="35.56" y2="12.7" width="0.4064" layer="1"/>
+<wire x1="21.59" y1="12.7" x2="31.75" y2="12.7" width="0.4064" layer="1"/>
+<wire x1="31.75" y1="12.7" x2="34.29" y2="15.24" width="0.4064" layer="1"/>
+<wire x1="34.29" y1="15.24" x2="35.56" y2="15.24" width="0.4064" layer="1"/>
+<wire x1="35.56" y1="15.24" x2="38.735" y2="15.24" width="0.4064" layer="1"/>
+<wire x1="38.735" y1="15.24" x2="40.005" y2="13.97" width="0.4064" layer="1"/>
+<wire x1="40.005" y1="13.97" x2="40.005" y2="12.7" width="0.4064" layer="1"/>
 </signal>
 <signal name="GND">
@@
 <contactref element="R1" pad="1"/>
 <contactref element="JP2" pad="3"/>
-<wire x1="31.75" y1="5.08" x2="35.56" y2="5.08" width="0.4064" layer="16"/>
-<wire x1="35.56" y1="5.08" x2="38.1" y2="5.08" width="0.4064" layer="16"/>
-<wire x1="38.1" y1="5.08" x2="40.005" y2="6.985" width="0.4064" layer="16"/>
-<wire x1="40.005" y1="6.985" x2="40.005" y2="7.62" width="0.4064" layer="16"/>
-<wire x1="35.56" y1="8.89" x2="35.56" y2="5.08" width="0.4064" layer="16"/>
-<wire x1="31.75" y1="5.08" x2="29.21" y2="2.54" width="0.4064" layer="1"/>
-<wire x1="29.21" y1="2.54" x2="7.62" y2="2.54" width="0.4064" layer="1"/>
+<wire x1="40.005" y1="6.985" x2="40.005" y2="7.62" width="0" layer="19" extent="1-16"/>
+<wire x1="35.56" y1="2.54" x2="31.75" y2="2.54" width="0.4064" layer="1"/>
+<wire x1="31.75" y1="2.54" x2="7.62" y2="2.54" width="0.4064" layer="1"/>
 <wire x1="7.62" y1="2.54" x2="3.81" y2="6.35" width="0.4064" layer="1"/>
 <wire x1="3.81" y1="6.35" x2="3.81" y2="7.62" width="0.4064" layer="1"/>
+<contactref element="C2" pad="2"/>
+<wire x1="31.75" y1="5.08" x2="31.75" y2="2.54" width="0.4064" layer="1"/>
+<wire x1="35.56" y1="12.7" x2="35.56" y2="10.16" width="0.4064" layer="16"/>
+<wire x1="35.56" y1="10.16" x2="38.1" y2="7.62" width="0.4064" layer="16"/>
+<wire x1="38.1" y1="7.62" x2="40.005" y2="7.62" width="0.4064" layer="16"/>
+<wire x1="35.56" y1="2.54" x2="38.1" y2="2.54" width="0.4064" layer="1"/>
+<wire x1="38.1" y1="2.54" x2="40.005" y2="4.445" width="0.4064" layer="1"/>
+<wire x1="40.005" y1="7.62" x2="40.005" y2="4.445" width="0.4064" layer="1"/>
 </signal>
 <signal name="SIG">
 <contactref element="R3" pad="2"/>
 <contactref element="JP1" pad="2"/>
-<wire x1="31.75" y1="10.16" x2="40.005" y2="10.16" width="0.4064" layer="1"/>
+<wire x1="31.75" y1="10.16" x2="35.56" y2="10.16" width="0.4064" layer="1"/>
+<contactref element="C2" pad="1"/>
+<wire x1="35.56" y1="10.16" x2="40.005" y2="10.16" width="0.4064" layer="1"/>
+<wire x1="35.56" y1="5.08" x2="35.56" y2="10.16" width="0.4064" layer="1"/>
 </signal>
 <signal name="N$1">
@@
 <contactref element="T1" pad="C"/>
 <contactref element="R3" pad="1"/>
-<wire x1="26.67" y1="10.16" x2="26.67" y2="5.08" width="0.4064" layer="16"/>
-<wire x1="26.67" y1="10.16" x2="24.13" y2="7.62" width="0.4064" layer="16"/>
-<wire x1="24.13" y1="7.62" x2="21.59" y2="7.62" width="0.4064" layer="16"/>
+<wire x1="26.67" y1="10.16" x2="26.67" y2="7.62" width="0.4064" layer="16"/>
+<wire x1="26.67" y1="7.62" x2="26.67" y2="5.08" width="0.4064" layer="16"/>
+<wire x1="21.59" y1="7.62" x2="26.67" y2="7.62" width="0.4064" layer="16"/>
 </signal>
 <signal name="N$2">
@@
 <contactref element="JP2" pad="2"/>
 <contactref element="R4" pad="2"/>
-<wire x1="3.81" y1="10.16" x2="7.62" y2="10.16" width="0.4064" layer="1"/>
+<wire x1="3.81" y1="10.16" x2="6.35" y2="10.16" width="0.4064" layer="1"/>
 </signal>
 <signal name="N$7">
 <contactref element="R4" pad="1"/>
 <contactref element="JP3" pad="1"/>
-<wire x1="12.7" y1="10.16" x2="15.24" y2="10.16" width="0.4064" layer="1"/>
+<wire x1="11.43" y1="10.16" x2="13.97" y2="10.16" width="0.4064" layer="1"/>
 </signal>
 </signals>
